Commit message: 2WD_Front_DiffDrive_NoRearSteer

File: src/car_body/description/car.xacro (robot description, xacro)
@@ -1,13 +1,28 @@
 <?xml version="1.0"?>
-<robot xmlns:xacro="http://www.ros.org/wiki/xacro" name="robot">
-    <xacro:include filename="color.urdf.xacro" />
-    <xacro:include filename="inertial_macros.urdf.xacro" />
-    <link name="world"></link>
+<robot xmlns:xacro="http://www.ros.org/wiki/xacro">
+    <xacro:include filename="inertial_macros.xacro" />
+    <material name="white">
+        <color rgba="1 1 1 1" />
+    </material>
+    <material name="orange">
+        <color rgba="1 0.3 0.1 1" />
+    </material>
+    <material name="blue">
+        <color rgba="0.2 0.2 1 1" />
+    </material>
+    <material name="black">
+        <color rgba="0 0 0 1" />
+    </material>
+    <material name="red">
+        <color rgba="1 0 0 1" />
+    </material>
+    <link name="base_link">
+    </link>
     <joint name="chassis_joint" type="fixed">
-        <parent link="world" />
-        <child link="chassis_link" />
+        <parent link="base_link" />
+        <child link="chassis" />
         <origin xyz="-0.1 0 0" />
     </joint>
-    <link name="chassis_link">
+    <link name="chassis">
         <visual>
             <origin xyz="0.21 0 0.08" />
@@ -23,21 +38,21 @@
             </geometry>
         </collision>
-        <xacro_inertial_box mass="8" x="0.42" y="0.22" z="0.16">
+        <xacro:inertial_box mass="8" x="0.42" y="0.22" z="0.16">
             <origin xyz="0.21 0 0.08" rpy="0 0 0" />
-        </xacro_inertial_box>
+        </xacro:inertial_box>
     </link>
+    <gazebo reference="chassis">
+        <material>Gazebo/Red</material>
+    </gazebo>
     <joint
         name="front_left_wheel_joint" type="continuous">
-        <parent link="world" />
-        <child link="front_left_wheel_link" />
-        <origin xyz="0.22 0.11 0" rpy="-${pi/2} 0 0" />
+        <parent link="base_link" />
+        <child link="front_left_wheel" />
+        <origin xyz="0.22 0.15 0" rpy="-${pi/2} 0 0" />
         <axis xyz="0 0 1" />
-        <ackermann_steering_controller />
-        <steer_angle>0.2</steer_angle>
-        <wheelbase>1.0</wheelbase>
-        <track_width>0.8</track_width>
+        <limit lower="-3.1416" upper="3.1416" effort="100" velocity="3.0" />
     </joint>
     <link
-        name="front_left_wheel_link">
+        name="front_left_wheel">
         <visual>
             <geometry>
@@ -51,21 +66,21 @@
             </geometry>
         </collision>
-        <inertial_cylinder mass="0.8" length="0.06" radius="0.04">
+        <xacro:inertial_cylinder mass="0.8" length="0.06" radius="0.04">
             <origin xyz="0 0 0" rpy="0 0 0" />
-        </inertial_cylinder>
+        </xacro:inertial_cylinder>
     </link>
+    <gazebo reference="front_left_wheel">
+        <material>Gazebo/Black</material>
+    </gazebo>
     <joint
         name="front_right_wheel_joint" type="continuous">
-        <parent link="world" />
-        <child link="front_right_wheel_link" />
-        <origin xyz="0.22 -0.11 0" rpy="${pi/2} 0 0" />
+        <parent link="base_link" />
+        <child link="front_right_wheel" />
+        <origin xyz="0.22 -0.15 0" rpy="${pi/2} 0 0" />
         <axis xyz="0 0 -1 " />
-        <ackermann_steering_controller />
-        <steer_angle>-1</steer_angle>
-        <wheelbase>1.0</wheelbase>
-        <track_width>0.8</track_width>
+        <limit lower="-3.1416" upper="3.1416" effort="100" velocity="3.0" />
     </joint>
     <link
-        name="front_right_wheel_link">
+        name="front_right_wheel">
         <visual>
             <geometry>
@@ -79,17 +94,20 @@
             </geometry>
         </collision>
-        <inertial_cylinder mass="0.8" length="0.06" radius="0.04">
+        <xacro:inertial_cylinder mass="0.8" length="0.06" radius="0.04">
             <origin xyz="0 0 0" rpy="0 0 0" />
-        </inertial_cylinder>
+        </xacro:inertial_cylinder>
     </link>
+    <gazebo reference="front_right_wheel">
+        <material>Gazebo/Black</material>
+    </gazebo>
     <joint
         name="rear_left_wheel_joint" type="continuous">
-        <parent link="world" />
-        <child link="rear_left_wheel_link" />
-        <origin xyz="0 0.11 0" rpy="-${pi/2} 0 0" />
+        <parent link="base_link" />
+        <child link="rear_left_wheel" />
+        <origin xyz="0 0.15 0" rpy="-${pi/2} 0 0" />
         <axis xyz="0 0 1" />
     </joint>
     <link
-        name="rear_left_wheel_link">
+        name="rear_left_wheel">
         <visual>
             <geometry>
@@ -103,17 +121,20 @@
             </geometry>
         </collision>
-        <inertial_cylinder mass="0.8" length="0.06" radius="0.04">
+        <xacro:inertial_cylinder mass="0.8" length="0.06" radius="0.04">
             <origin xyz="0 0 0" rpy="0 0 0" />
-        </inertial_cylinder>
+        </xacro:inertial_cylinder>
     </link>
+    <gazebo reference="rear_left_wheel">
+        <material>Gazebo/Black</material>
+    </gazebo>
     <joint
         name="rear_right_wheel_joint" type="continuous">
-        <parent link="world" />
-        <child link="rear_right_wheel_link" />
-        <origin xyz="0 -0.11 0" rpy="${pi/2} 0 0" />
+        <parent link="base_link" />
+        <child link="rear_right_wheel" />
+        <origin xyz="0 -0.15 0" rpy="${pi/2} 0 0" />
         <axis xyz="0 0 -1 " />
     </joint>
     <link
-        name="rear_right_wheel_link">
+        name="rear_right_wheel">
         <visual>
             <geometry>
@@ -127,7 +148,10 @@
             </geometry>
         </collision>
-        <inertial_cylinder mass="0.8" length="0.06" radius="0.04">
+        <xacro:inertial_cylinder mass="0.8" length="0.06" radius="0.04">
             <origin xyz="0 0 0" rpy="0 0 0" />
-        </inertial_cylinder>
+        </xacro:inertial_cylinder>
     </link>
+    <gazebo reference="rear_right_wheel">
+        <material>Gazebo/Black</material>
+    </gazebo>
 </robot>

Commit message: Car Body URDF modified

File: src/car_body/description/car.xacro (robot description, xacro)
@@ -2,4 +2,11 @@
 <robot xmlns:xacro="http://www.ros.org/wiki/xacro">
     <xacro:include filename="inertial_macros.xacro" />
+    <xacro:arg name="car_controller_yaml_file"
+        default="$(find car_gazebo)/config/ackermann_controller.yaml" />
+    <xacro:property name="bearing_friction_coeff" value="0.0015" />
+    <xacro:property name="wheel_joint_damping" value="10" />
+    <xacro:property name="steering_joint_damping" value="20" />
+    <xacro:property name="gravity" value="9.81" />
+    <xacro:property name="chassis_mass" value="8.0" />
     <material name="white">
         <color rgba="1 1 1 1" />
@@ -19,25 +26,39 @@
     <link name="base_link">
     </link>
+    <inertial>
+        <mass value="0.01" />
+        <inertia ixx="1.0" ixy="0.0" ixz="0.0" iyy="1.0" iyz="0.0" izz="1.0" />
+    </inertial>
+    <joint name="base_joint" type="fixed">
+        <parent link="base_link" />
+        <child link="base_footprint" />
+        <origin xyz="0 0 -0.1" />
+    </joint>
+    <link name="base_footprint">
+    </link>
+    <inertial>
+        <mass value="0.01" />
+        <inertia ixx="1.0" ixy="0.0" ixz="0.0" iyy="1.0" iyz="0.0" izz="1.0" />
+    </inertial>
     <joint name="chassis_joint" type="fixed">
-        <parent link="base_link" />
-        <child link="chassis" />
-        <origin xyz="-0.1 0 0" />
+        <parent link="base_link"></parent>
+        <child link="chassis"></child>
     </joint>
     <link name="chassis">
         <visual>
-            <origin xyz="0.21 0 0.08" />
-            <geometry>
-                <box size="0.42 0.22 0.16" />
+            <origin xyz="0.5 0 0.25" />
+            <geometry>
+                <box size="1 0.55 0.45" />
             </geometry>
             <material name="red" />
         </visual>
         <collision>
-            <origin xyz="0.21 0 0.08" />
-            <geometry>
-                <box size="0.42 0.22 0.16" />
-            </geometry>
-        </collision>
-        <xacro:inertial_box mass="8" x="0.42" y="0.22" z="0.16">
-            <origin xyz="0.21 0 0.08" rpy="0 0 0" />
+            <origin xyz="0.5 0 0.25" />
+            <geometry>
+                <box size="1 0.55 0.45" />
+            </geometry>
+        </collision>
+        <xacro:inertial_box mass="8" x="1" y="0.55" z="0.45">
+            <origin xyz="0.5 0 0.25" rpy="0 0 0" />
         </xacro:inertial_box>
     </link>
@@ -45,11 +66,26 @@
         <material>Gazebo/Red</material>
     </gazebo>
-    <joint
-        name="front_left_wheel_joint" type="continuous">
-        <parent link="base_link" />
+    <!-- Left Steering Joint -->
+    <joint
+        name="left_steering_joint" type="revolute">
+        <parent link="base_link" />
+        <child link="left_steering_link" />
+        <origin xyz="0.75 0.225 0" />
+        <axis xyz="0 0 1" />
+        <limit effort="100" lower="-0.523" upper="0.523" velocity="0.5" />
+        <dynamics damping="${steering_joint_damping}"
+            friction="${bearing_friction_coeff*gravity*chassis_mass}" />
+    </joint>
+    <link name="left_steering_link">
+        <inertial>
+            <mass value="0.001" />
+            <inertia ixx="1.0" ixy="0.0" ixz="0.0" iyy="1.0" iyz="0.0" izz="1.0" />
+        </inertial>
+    </link>
+    <joint name="front_left_wheel_joint" type="continuous">
+        <parent link="left_steering_link" />
         <child link="front_left_wheel" />
-        <origin xyz="0.22 0.15 0" rpy="-${pi/2} 0 0" />
-        <axis xyz="0 0 1" />
-        <limit lower="-3.1416" upper="3.1416" effort="100" velocity="3.0" />
+        <origin xyz="0 0.05 0" rpy="-${pi/2} 0 0" />
+        <axis xyz="0 0 1" />
     </joint>
     <link
@@ -57,11 +93,53 @@
         <visual>
             <geometry>
-                <cylinder length="0.06" radius="0.04" />
-            </geometry>
-            <material name="black" />
-        </visual>
-        <collision>
-            <geometry>
-                <cylinder length="0.06" radius="0.04" />
+                <cylinder length="0.08" radius="0.115" />
+            </geometry>
+            <material name="black" />
+        </visual>
+        <collision>
+            <geometry>
+                <cylinder length="0.08" radius="0.115" />
+            </geometry>
+        </collision>
+        <xacro:inertial_cylinder mass="0.8" length="0.08" radius="0.115">
+            <origin xyz="0 0 0" rpy="0 0 0" />
+        </xacro:inertial_cylinder>
+    </link>
+    <gazebo reference="front_left_wheel">
+        <material>Gazebo/Black</material>
+    </gazebo>
+    <joint
+        name="right_steering_joint" type="revolute">
+        <parent link="base_link" />
+        <child link="right_steering_link" />
+        <origin xyz="0.75 -0.225 0" />
+        <axis xyz="0 0 1 " />
+        <limit effort="1000.0" lower="-0.523" upper="0.523" velocity="0.5" />
+        <dynamics damping="${steering_joint_damping}"
+            friction="${bearing_friction_coeff*gravity*chassis_mass}" />
+    </joint>
+    <link name="right_steering_link">
+        <inertial>
+            <mass value="0.001" />
+            <inertia ixx="1.0" ixy="0.0" ixz="0.0" iyy="1.0" iyz="0.0" izz="1.0" />
+        </inertial>
+    </link>
+    <joint name="front_right_wheel_joint" type="continuous">
+        <parent link="right_steering_link" />
+        <child link="front_right_wheel" />
+        <origin xyz="0 -0.05 0" rpy="-${pi/2} 0 0" />
+        <axis xyz="0 0 1" />
+    </joint>
+    <link
+        name="front_right_wheel">
+        <visual>
+            <geometry>
+                <cylinder length="0.08" radius="0.115" />
+            </geometry>
+            <material name="black" />
+        </visual>
+        <collision>
+            <geometry>
+                <cylinder length="0.08" radius="0.115" />
             </geometry>
         </collision>
@@ -70,26 +148,52 @@
         </xacro:inertial_cylinder>
     </link>
-    <gazebo reference="front_left_wheel">
-        <material>Gazebo/Black</material>
-    </gazebo>
-    <joint
-        name="front_right_wheel_joint" type="continuous">
-        <parent link="base_link" />
-        <child link="front_right_wheel" />
-        <origin xyz="0.22 -0.15 0" rpy="${pi/2} 0 0" />
+    <gazebo reference="front_right_wheel">
+        <material>Gazebo/Black</material>
+    </gazebo>
+    <joint
+        name="rear_left_wheel_joint" type="continuous">
+        <parent link="base_link" />
+        <child link="rear_left_wheel" />
+        <origin xyz="0.22 0.275 0" rpy="-${pi/2} 0 0" />
+        <axis xyz="0 0 1" />
+    </joint>
+    <link
+        name="rear_left_wheel">
+        <visual>
+            <geometry>
+                <cylinder length="0.08" radius="0.115" />
+            </geometry>
+            <material name="black" />
+        </visual>
+        <collision>
+            <geometry>
+                <cylinder length="0.08" radius="0.115" />
+            </geometry>
+        </collision>
+        <xacro:inertial_cylinder mass="0.8" length="0.06" radius="0.04">
+            <origin xyz="0 0 0" rpy="0 0 0" />
+        </xacro:inertial_cylinder>
+    </link>
+    <gazebo reference="rear_left_wheel">
+        <material>Gazebo/Black</material>
+    </gazebo>
+    <joint
+        name="rear_right_wheel_joint" type="continuous">
+        <parent link="base_link" />
+        <child link="rear_right_wheel" />
+        <origin xyz="0.22 -0.275 0" rpy="${pi/2} 0 0" />
         <axis xyz="0 0 -1 " />
-        <limit lower="-3.1416" upper="3.1416" effort="100" velocity="3.0" />
-    </joint>
-    <link
-        name="front_right_wheel">
-        <visual>
-            <geometry>
-                <cylinder length="0.06" radius="0.04" />
-            </geometry>
-            <material name="black" />
-        </visual>
-        <collision>
-            <geometry>
-                <cylinder length="0.06" radius="0.04" />
+    </joint>
+    <link
+        name="rear_right_wheel">
+        <visual>
+            <geometry>
+                <cylinder length="0.08" radius="0.115" />
+            </geometry>
+            <material name="black" />
+        </visual>
+        <collision>
+            <geometry>
+                <cylinder length="0.08" radius="0.115" />
             </geometry>
         </collision>
@@ -98,60 +202,41 @@
         </xacro:inertial_cylinder>
     </link>
-    <gazebo reference="front_right_wheel">
-        <material>Gazebo/Black</material>
-    </gazebo>
-    <joint
-        name="rear_left_wheel_joint" type="continuous">
-        <parent link="base_link" />
-        <child link="rear_left_wheel" />
-        <origin xyz="0 0.15 0" rpy="-${pi/2} 0 0" />
-        <axis xyz="0 0 1" />
-    </joint>
-    <link
-        name="rear_left_wheel">
-        <visual>
-            <geometry>
-                <cylinder length="0.06" radius="0.04" />
-            </geometry>
-            <material name="black" />
-        </visual>
-        <collision>
-            <geometry>
-                <cylinder length="0.06" radius="0.04" />
-            </geometry>
-        </collision>
-        <xacro:inertial_cylinder mass="0.8" length="0.06" radius="0.04">
-            <origin xyz="0 0 0" rpy="0 0 0" />
-        </xacro:inertial_cylinder>
-    </link>
-    <gazebo reference="rear_left_wheel">
-        <material>Gazebo/Black</material>
-    </gazebo>
-    <joint
-        name="rear_right_wheel_joint" type="continuous">
-        <parent link="base_link" />
-        <child link="rear_right_wheel" />
-        <origin xyz="0 -0.15 0" rpy="${pi/2} 0 0" />
-        <axis xyz="0 0 -1 " />
-    </joint>
-    <link
-        name="rear_right_wheel">
-        <visual>
-            <geometry>
-                <cylinder length="0.06" radius="0.04" />
-            </geometry>
-            <material name="black" />
-        </visual>
-        <collision>
-            <geometry>
-                <cylinder length="0.06" radius="0.04" />
-            </geometry>
-        </collision>
-        <xacro:inertial_cylinder mass="0.8" length="0.06" radius="0.04">
-            <origin xyz="0 0 0" rpy="0 0 0" />
-        </xacro:inertial_cylinder>
-    </link>
     <gazebo reference="rear_right_wheel">
         <material>Gazebo/Black</material>
     </gazebo>
+    <!-- Ackermann driver -->
+    <ros2_control name="GazeboSystem" type="system">
+        <!-- the name of the hardware interface plugin to load -->
+        <hardware>
+            <plugin>gazebo_ros2_control/GazeboSystem</plugin>
+        </hardware>
+        <!-- talks to these joints of the car -->
+        <joint name="rear_left_wheel_joint">
+            <command_interface name="velocity" />
+            <state_interface name="position" />
+            <state_interface name="velocity" />
+        </joint>
+        <joint name="rear_right_wheel_joint">
+            <command_interface name="velocity" />
+            <state_interface name="position" />
+            <state_interface name="velocity" />
+        </joint>
+        <joint name="left_steering_joint">
+            <command_interface name="position" />
+            <state_interface name="position" />
+            <state_interface name="velocity" />
+        </joint>
+        <joint name="right_steering_joint">
+            <command_interface name="position" />
+            <state_interface name="position" />
+            <state_interface name="velocity" />
+        </joint>
+    </ros2_control>
+    <gazebo>
+        <plugin filename="libgazebo_ros2_control.so" name="gazebo_ros2_control">
+            <robot_param>robot_description</robot_param>
+            <robot_param_node>robot_state_publisher</robot_param_node>
+            <parameters>$(arg car_controller_yaml_file)</parameters>
+        </plugin>
+    </gazebo>
 </robot>

File: src/car_body/description/vehicle.urdf.xacro (robot description, xacro)
@@ -2,4 +2,5 @@
 <robot xmlns:xacro="http://www.ros.org/wiki/xacro" name="robot">
     <xacro:include filename="car.xacro" />
-    <xacro:include filename="gazebo_control.xacro" />
+    <!-- <xacro:include filename="gazebo_control.xacro" /> -->
+    <xacro:include filename="lidar.xacro" />
 </robot>
