Commit message: lidar urdf setup

File: src/car_gazebo/urdf/car.urdf.xacro (robot description, xacro)
@@ -6,6 +6,6 @@
         <xacro:property name="base_mass" value="8.0" /> <!-- arbitrary value for base mass -->
         <xacro:property name="base_length" value="1.0" />
-        <xacro:property name="base_width" value="0.55" />
-        <xacro:property name="base_height" value="0.45" />
+        <xacro:property name="base_width" value="0.53" />
+        <xacro:property name="base_height" value="0.32" />
         <xacro:property name="wheel_mass" value="0.1" /> <!-- arbitrary value for wheel mass -->
         <xacro:property name="wheelbase" value="0.54" />

File: src/car_gazebo/urdf/car_ros2_control.xacro (robot description, xacro)
@@ -19,3 +19,8 @@
     </ros2_control>
   </xacro:macro>
+  <gazebo>
+    <plugin name="gazebo_ros2_control" filename="libgazebo_ros2_control.so">
+      <parameters>$(find car_gazebo)/config/carlikebot_controllers.yaml</parameters>
+    </plugin>
+  </gazebo>
 </robot>

File: src/car_gazebo/urdf/vehicle.urdf.xacro (robot description, xacro)
@@ -5,6 +5,6 @@
   <xacro:include filename="car.urdf.xacro" />
   <xacro:include filename="car_ros2_control.xacro" />
+  <xacro:include filename="car_lidar.xacro" />
   <xacro:carlikebot prefix="$(arg prefix)" />
-  <xacro:carlikebot_ros2_control
-    name="CarlikeBot" prefix="$(arg prefix)" />
+  <xacro:carlikebot_ros2_control name="CarlikeBot" prefix="$(arg prefix)" />
 </robot>

Commit message: odom rotating problem, urdf reconfigure, stm to ros setup

File: src/car_gazebo/urdf/car.urdf.xacro (robot description, xacro)
@@ -9,5 +9,5 @@
         <xacro:property name="base_height" value="0.32" />
         <xacro:property name="wheel_mass" value="0.1" /> <!-- arbitrary value for wheel mass -->
-        <xacro:property name="wheelbase" value="0.54" />
+        <xacro:property name="wheelbase" value="0.46" />
         <xacro:property name="wheel_len" value="0.08" />
         <xacro:property name="wheel_radius" value="0.115" />
@@ -98,5 +98,5 @@
             <axis xyz="1 0 0" />
             <limit effort="100.0" velocity="100.0" />
-            <dynamics damping="0.2" />
+            <!-- <dynamics damping="0.2" /> -->
         </joint>
         <!-- rear right wheel -->
@@ -130,5 +130,5 @@
             <axis xyz="1 0 0" />
             <limit effort="100.0" velocity="100.0" />
-            <dynamics damping="0.2" />
+            <!-- <dynamics damping="0.2" /> -->
             <mimic joint="${prefix}virtual_rear_wheel_joint" multiplier="1.0" offset="0.0" />
         </joint>
@@ -163,5 +163,5 @@
             <axis xyz="1 0 0" />
             <limit effort="100.0" velocity="100.0" />
-            <dynamics damping="0.2" />
+            <!-- <dynamics damping="0.2" /> -->
             <mimic joint="${prefix}virtual_rear_wheel_joint" multiplier="1.0" offset="0.0" />
         </joint>
@@ -182,6 +182,6 @@
             <origin xyz="${wheelbase/2} 0 -${base_height/2}" rpy="0 0 ${PI/2}" />
             <axis xyz="0 0 1" />
-            <limit lower="-0.4" upper="0.4" effort="100.0" velocity="0.0" />
-            <dynamics damping="0.2" />
+            <limit lower="-0.3488" upper="0.3488" effort="100.0" velocity="0.0" />
+            <!-- <dynamics damping="0.2" /> -->
         </joint>
         <!-- front right wheel -->
@@ -214,6 +214,6 @@
             <origin xyz="${wheelbase/2} ${base_width/2} -${base_height/2}" rpy="0 0 ${PI/2}" />
             <axis xyz="0 0 1" />
-            <limit lower="-0.4" upper="0.4" effort="100.0" velocity="0.0" />
-            <dynamics damping="0.2" />
+            <limit lower="-0.3488" upper="0.3488" effort="100.0" velocity="0.0" />
+            <!-- <dynamics damping="0.2" /> -->
             <mimic joint="${prefix}virtual_front_wheel_joint" multiplier="1.0" offset="0.0" />
         </joint>
@@ -247,6 +247,6 @@
             <origin xyz="${wheelbase/2} -${base_width/2} -${base_height/2}" rpy="0 0 ${PI/2}" />
             <axis xyz="0 0 1" />
-            <limit lower="-0.4" upper="0.4" effort="100.0" velocity="0.0" />
-            <dynamics damping="0.2" />
+            <limit lower="-0.3488" upper="0.3488" effort="100.0" velocity="0.0" />
+            <!-- <dynamics damping="0.2" /> -->
             <mimic joint="${prefix}virtual_front_wheel_joint" multiplier="1.0" offset="0.0" />
         </joint>

File: src/car_gazebo/urdf/car_ros2_control.xacro (robot description, xacro)
@@ -19,8 +19,8 @@
     </ros2_control>
   </xacro:macro>
-  <gazebo>
+  <!-- <gazebo>
     <plugin name="gazebo_ros2_control" filename="libgazebo_ros2_control.so">
       <parameters>$(find car_gazebo)/config/carlikebot_controllers.yaml</parameters>
     </plugin>
-  </gazebo>
+  </gazebo> -->
 </robot>
