Commit message: imu, lidar frame and map, odom, baselink transformation done

File: src/car_gazebo/urdf/imu.urdf.xacro (robot description, xacro)
@@ -19,5 +19,5 @@
         </inertial>
     </xacro:macro>
-    <link name="imu_link">
+    <link name="imu_frame">
         <visual>
             <geometry>
@@ -38,5 +38,5 @@
     <joint name="imu_joint" type="fixed">
         <parent link="chassis_link" />
-        <child link="imu_link" />
+        <child link="imu_frame" />
         <origin xyz="-0.13 -0.01 0.18" rpy="0 0 0" />
     </joint>

Commit message: 2D Goal Pose: better map, filtered odom from from bno and ros2_odom with high covariance, nav2 params, imu urdf rewrite, teleop

File: src/car_gazebo/urdf/imu.urdf.xacro (robot description, xacro)
@@ -39,5 +39,5 @@
         <parent link="chassis_link" />
         <child link="imu_frame" />
-        <origin xyz="-0.13 -0.01 0.18" rpy="0 0 0" />
+        <origin xyz="-0.20 0.11 -0.02" rpy="0 0 0" />
     </joint>
 </robot>
